Commit message: First Commit2

File: description/robot_core.xacro (robot description, xacro)
@@ -43,6 +43,6 @@
     <parent link="base_link"/>
     <child link="left_wheel"/>
-    <origin xyz="0 0.4 -0.05" rpy="-${pi/2} 0 0"/>
-    <axis xyz="0 0.5 1"/>
+    <origin xyz="0 0.375 -0.15" rpy="-${pi/2} 0 0"/>
+    <axis xyz="0 0 1"/>
 </joint>
 <link name="left_wheel">
@@ -67,6 +67,6 @@
     <parent link="base_link"/>
     <child link="right_wheel"/>
-    <origin xyz="0 -0.4 -0.05" rpy="${pi/2} 0 0"/>
-    <axis xyz="0 0.5 -1"/>
+    <origin xyz="0 -0.375 -0.15" rpy="${pi/2} 0 0"/>
+    <axis xyz="0 0 -1"/>
 </joint>
 <link name="right_wheel">

Commit message: First Commit3

File: description/robot_core.xacro (robot description, xacro)
@@ -39,9 +39,12 @@
     </xacro:inertial_box>
 </link>
+<gazebo reference="chassis">
+    <material>Gazebo/White</material>
+</gazebo>
 <!-- LEFT WHEEL -->
 <joint name="left_wheel_joint" type="continuous">
     <parent link="base_link"/>
     <child link="left_wheel"/>
-    <origin xyz="0 0.375 -0.15" rpy="-${pi/2} 0 0"/>
+    <origin xyz="-0.35 0.375 -0.12" rpy="-${pi/2} 0 0"/>
     <axis xyz="0 0 1"/>
 </joint>
@@ -63,9 +66,39 @@
     </xacro:inertial_cylinder>
 </link>
+<gazebo reference="left_wheel">
+    <material>Gazebo/Blue</material>
+</gazebo>
+<!-- FRONT LEFT WHEEL -->
+<joint name="front_left_wheel_joint" type="continuous">
+    <parent link="base_link"/>
+    <child link="front_left_wheel"/>
+    <origin xyz="0.45 0.375 -0.12" rpy="-${pi/2} 0 0"/>
+    <axis xyz="0 0 1"/>
+</joint>
+<link name="front_left_wheel">
+    <visual>
+        <geometry>
+            <cylinder length="0.06" radius="0.15" />
+        </geometry>
+        <material name="blue"/>
+    </visual>
+     <collision>
+        <geometry>
+            <cylinder length="0.06" radius="0.15" />
+        </geometry>
+        <material name="blue"/>
+    </collision>
+    <xacro:inertial_cylinder mass="0.1" length="0.06" radius="0.15">
+        <origin xyz="0 0 0" rpy="0 0 0"/>
+    </xacro:inertial_cylinder>
+</link>
+<gazebo reference="front_left_wheel">
+    <material>Gazebo/Blue</material>
+</gazebo>
 <!-- RIGHT WHEEL -->
 <joint name="right_wheel_joint" type="continuous">
     <parent link="base_link"/>
     <child link="right_wheel"/>
-    <origin xyz="0 -0.375 -0.15" rpy="${pi/2} 0 0"/>
+    <origin xyz="-0.35 -0.375 -0.12" rpy="${pi/2} 0 0"/>
     <axis xyz="0 0 -1"/>
 </joint>
@@ -87,4 +120,34 @@
     </xacro:inertial_sphere>
 </link>
+<gazebo reference="right_wheel">
+    <material>Gazebo/Blue</material>
+</gazebo>
+<!-- RIGHT WHEEL -->
+<joint name="front_right_wheel_joint" type="continuous">
+    <parent link="base_link"/>
+    <child link="front_right_wheel"/>
+    <origin xyz="0.45 -0.375 -0.12" rpy="${pi/2} 0 0"/>
+    <axis xyz="0 0 -1"/>
+</joint>
+<link name="front_right_wheel">
+    <visual>
+        <geometry>
+            <cylinder length="0.06" radius="0.15" />
+        </geometry>
+        <material name="blue"/>
+    </visual>
+    <collision>
+        <geometry>
+            <cylinder length="0.06" radius="0.15" />
+        </geometry>
+        <material name="blue"/>
+    </collision>
+    <xacro:inertial_sphere mass="0.1" radius="0.15">
+        <origin xyz="0 -0.4 -0.05" rpy="0 0 0"/>
+    </xacro:inertial_sphere>
+</link>
+<gazebo reference="front_right_wheel">
+    <material>Gazebo/Blue</material>
+</gazebo>
 <!-- CASTER WHEEL -->
 <joint name="caster_wheel_joint" type="fixed">
@@ -107,3 +170,8 @@
     </collision>
 </link>
+<gazebo reference="caster_wheel">
+    <material>Gazebo/Black</material>
+    <mu1 value="0.001"/>
+    <mu2 value="0.001"/>
+</gazebo>
 </robot>
