Commit message: Pending changes exported from your codespace

File: description/gazebo_control.xacro (robot description, xacro)
@@ -2,10 +2,14 @@
 <robot xmlns:xacro="http://www.ros.org/wiki/xacro">
     <gazebo>
-        <plugin name='diff_drive' filename='libgazebo_ros_diff_drive.so'>
+        <plugin name="diff_drive" filename="libgazebo_ros_diff_drive.so">
             <!-- Wheel Information -->
+            <left_joint>left_front_wheel_joint</left_joint>  <!-- Reference to the left front wheel joint -->
+            <right_joint>right_front_wheel_joint</right_joint>  <!-- Reference to the right front wheel joint -->
+            <wheel_separation>0.75</wheel_separation>  <!-- This can be adjusted to match your robot's wheelbase -->
+            <wheel_diameter>0.17</wheel_diameter>  <!-- Updated to match the wheel radius (2 * 0.085) -->
             <left_joint>left_wheel_joint</left_joint>
             <right_joint>right_wheel_joint</right_joint>
-            <wheel_separation>0.35</wheel_separation>
-            <wheel_diameter>0.1</wheel_diameter>
+            <wheel_separation>0.75</wheel_separation>
+            <wheel_diameter>0.17</wheel_diameter>
             <!-- Limits -->
             <max_wheel_torque>200</max_wheel_torque>

File: description/robot.urdf.xacro (robot description, xacro)
@@ -1,5 +1,15 @@
 <?xml version="1.0"?>
 <robot xmlns:xacro="http://www.ros.org/wiki/xacro"  name="robot">
+    <xacro:arg name="use_ros2_control" default="true"/>
+    <xacro:arg name="sim_mode" default="false"/>
     <xacro:include filename="robot_core.xacro" />
-    <xacro:include filename="gazebo_control.xacro" />
+    <xacro:if value="$(arg use_ros2_control)">
+        <xacro:include filename="ros2_control.xacro" />
+    </xacro:if>
+    <xacro:unless value="$(arg use_ros2_control)">
+        <xacro:include filename="gazebo_control.xacro" />
+    </xacro:unless>
+    <xacro:include filename="lidar.xacro" />
+    <xacro:include filename="camera.xacro" />
+    <!-- <xacro:include filename="depth_camera.xacro" /> -->
 </robot>

File: description/robot_core.xacro (robot description, xacro)
@@ -1,177 +1,171 @@
 <?xml version="1.0"?>
 <robot xmlns:xacro="http://www.ros.org/wiki/xacro">
-<xacro:include filename="inertial_macros.xacro" />
+    <xacro:include filename="inertial_macros.xacro"/>
+    <xacro:property name="chassis_length" value="1.02"/>  <!-- Updated length -->
+    <xacro:property name="chassis_width" value="0.70"/>   <!-- Updated width -->
+    <xacro:property name="chassis_height" value="0.45"/>  <!-- Updated height -->
+    <xacro:property name="chassis_mass" value="1.0"/>
+    <xacro:property name="wheel_radius" value="0.085"/>   <!-- Updated wheel radius -->
+    <xacro:property name="wheel_thickness" value="0.05"/>  <!-- Updated wheel thickness -->
+    <xacro:property name="wheel_mass" value="0.05"/>
+    <xacro:property name="wheel_offset_x" value="0.51"/>   <!-- Updated offset for wheel placement -->
+    <xacro:property name="wheel_offset_y" value="0.375"/>   <!-- Updated offset for wheel placement -->
+    <xacro:property name="wheel_offset_z" value="0.0"/>    <!-- Height offset for wheels -->
     <material name="white">
-    <color rgba="1 1 1 1"/>
-</material>
-<material name="orange">
-    <color rgba="1 0.3 0.1 1"/>
-</material>
-<material name="blue">
-    <color rgba="0.2 0.2 1 1"/>
-</material>
-<material name="black">
-    <color rgba="0 0 0 1"/>
-</material>
-<link name="base_link">
-</link>
-<joint name="chassis_joint" type="fixed">
-    <parent link="base_link"/>
-    <child link="chassis"/>
-    <origin xyz="-0.1 0 0"/>
-</joint>
-<link name="chassis">
-    <visual>
-        <origin xyz="0.15 0 0.075" rpy="0 0 0"/>
-        <geometry>
-            <box size="0.9 0.7 0.45"/>
-        </geometry>
-        <material name="white"/>
-    </visual>
-    <collision>
-        <origin xyz="0.15 0 0.075" rpy="0 0 0"/>
-        <geometry>
-            <box size="0.9 0.7 0.45"/>
-        </geometry>
+        <color rgba="1 1 1 1" />
+    </material>
+    <material name="orange">
+        <color rgba="1 0.3 0.1 1"/>
+    </material>
+    <material name="blue">
+        <color rgba="0.2 0.2 1 1"/>
+    </material>
+    <material name="black">
+        <color rgba="0 0 0 1"/>
+    </material>
+    <material name="red">
+        <color rgba="1 0 0 1"/>
+    </material>
+    <!-- BASE LINK -->
+    <link name="base_link">
+    </link>
+    <!-- BASE_FOOTPRINT LINK -->
+    <joint name="base_footprint_joint" type="fixed">
+        <parent link="base_link"/>
+        <child link="base_footprint"/>
+        <origin xyz="0 0 0" rpy="0 0 0"/>
+    </joint>
+    <link name="base_footprint">
+    </link>
+    <!-- CHASSIS LINK -->
+    <joint name="chassis_joint" type="fixed">
+        <parent link="base_link"/>
+        <child link="chassis"/>
+        <origin xyz="${-wheel_offset_x} 0 ${-wheel_offset_z}"/>
+    </joint>
+    <link name="chassis">
+        <visual>
+            <origin xyz="${chassis_length/2} 0 ${chassis_height/2}"/>
+            <geometry>
+                <box size="${chassis_length} ${chassis_width} ${chassis_height}"/>
+            </geometry>
+            <material name="orange"/>
+        </visual>
+        <collision>
+            <origin xyz="${chassis_length/2} 0 ${chassis_height/2}"/>
+            <geometry>
+                <box size="${chassis_length} ${chassis_width} ${chassis_height}"/>
+            </geometry>
         </collision>
-    <xacro:inertial_box mass="0.5" x="0.9" y="0.7" z="0.45">
-        <origin xyz="0.15 0 0.075" rpy="0 0 0"/>
-    </xacro:inertial_box>
-</link>
-<gazebo reference="chassis">
-    <material>Gazebo/White</material>
-</gazebo>
-<!-- LEFT WHEEL -->
-<joint name="left_wheel_joint" type="continuous">
-    <parent link="base_link"/>
-    <child link="left_wheel"/>
-    <origin xyz="-0.35 0.375 -0.12" rpy="-${pi/2} 0 0"/>
-    <axis xyz="0 0 1"/>
-</joint>
-<link name="left_wheel">
-    <visual>
-        <geometry>
-            <cylinder length="0.06" radius="0.15" />
-        </geometry>
-        <material name="blue"/>
-    </visual>
-     <collision>
-        <geometry>
-            <cylinder length="0.06" radius="0.15" />
-        </geometry>
-        <material name="blue"/>
-    </collision>
-    <xacro:inertial_cylinder mass="0.1" length="0.06" radius="0.15">
-        <origin xyz="0 0 0" rpy="0 0 0"/>
-    </xacro:inertial_cylinder>
-</link>
-<gazebo reference="left_wheel">
-    <material>Gazebo/Blue</material>
-</gazebo>
-<!-- FRONT LEFT WHEEL -->
-<joint name="front_left_wheel_joint" type="continuous">
-    <parent link="base_link"/>
-    <child link="front_left_wheel"/>
-    <origin xyz="0.45 0.375 -0.12" rpy="-${pi/2} 0 0"/>
-    <axis xyz="0 0 1"/>
-</joint>
-<link name="front_left_wheel">
-    <visual>
-        <geometry>
-            <cylinder length="0.06" radius="0.15" />
-        </geometry>
-        <material name="blue"/>
-    </visual>
-     <collision>
-        <geometry>
-            <cylinder length="0.06" radius="0.15" />
-        </geometry>
-        <material name="blue"/>
-    </collision>
-    <xacro:inertial_cylinder mass="0.1" length="0.06" radius="0.15">
-        <origin xyz="0 0 0" rpy="0 0 0"/>
-    </xacro:inertial_cylinder>
-</link>
-<gazebo reference="front_left_wheel">
-    <material>Gazebo/Blue</material>
-</gazebo>
-<!-- RIGHT WHEEL -->
-<joint name="right_wheel_joint" type="continuous">
-    <parent link="base_link"/>
-    <child link="right_wheel"/>
-    <origin xyz="-0.35 -0.375 -0.12" rpy="${pi/2} 0 0"/>
-    <axis xyz="0 0 -1"/>
-</joint>
-<link name="right_wheel">
-    <visual>
-        <geometry>
-            <cylinder length="0.06" radius="0.15" />
-        </geometry>
-        <material name="blue"/>
-    </visual>
-    <collision>
-        <geometry>
-            <cylinder length="0.06" radius="0.15" />
-        </geometry>
-        <material name="blue"/>
-    </collision>
-    <xacro:inertial_sphere mass="0.1" radius="0.15">
-        <origin xyz="0 -0.4 -0.05" rpy="0 0 0"/>
-    </xacro:inertial_sphere>
-</link>
-<gazebo reference="right_wheel">
-    <material>Gazebo/Blue</material>
-</gazebo>
-<!-- RIGHT WHEEL -->
-<joint name="front_right_wheel_joint" type="continuous">
-    <parent link="base_link"/>
-    <child link="front_right_wheel"/>
-    <origin xyz="0.45 -0.375 -0.12" rpy="${pi/2} 0 0"/>
-    <axis xyz="0 0 -1"/>
-</joint>
-<link name="front_right_wheel">
-    <visual>
-        <geometry>
-            <cylinder length="0.06" radius="0.15" />
-        </geometry>
-        <material name="blue"/>
-    </visual>
-    <collision>
-        <geometry>
-            <cylinder length="0.06" radius="0.15" />
-        </geometry>
-        <material name="blue"/>
-    </collision>
-    <xacro:inertial_sphere mass="0.1" radius="0.15">
-        <origin xyz="0 -0.4 -0.05" rpy="0 0 0"/>
-    </xacro:inertial_sphere>
-</link>
-<gazebo reference="front_right_wheel">
-    <material>Gazebo/Blue</material>
-</gazebo>
-<!-- CASTER WHEEL -->
-<joint name="caster_wheel_joint" type="fixed">
-    <parent link="chassis"/>
-    <child link="caster_wheel"/>
-    <origin xyz="0.24 0 -0.2" rpy="0 0 0"/>
-</joint>
-<link name="caster_wheel">
-    <visual>
-        <geometry>
-            <sphere radius="0.08" />
-        </geometry>
-        <material name="black"/>
-    </visual>
-     <collision>
-        <geometry>
-            <sphere radius="0.08" />
-        </geometry>
-        <material name="black"/>
-    </collision>
-</link>
-<gazebo reference="caster_wheel">
-    <material>Gazebo/Black</material>
-    <mu1 value="0.001"/>
-    <mu2 value="0.001"/>
-</gazebo>
+        <xacro:inertial_box mass="0.5" x="${chassis_length}" y="${chassis_width}" z="${chassis_height}">
+            <origin xyz="${chassis_length/2} 0 ${chassis_height/2}" rpy="0 0 0"/>
+        </xacro:inertial_box>
+    </link>
+    <gazebo reference="chassis">
+        <material>Gazebo/Orange</material>
+    </gazebo>
+    <!-- LEFT FRONT WHEEL LINK -->
+    <joint name="left_front_wheel_joint" type="continuous">
+        <parent link="base_link"/>
+        <child link="left_front_wheel"/>
+        <origin xyz="${-wheel_offset_x} ${wheel_offset_y} 0" rpy="-${pi/2} 0 0"/>
+        <axis xyz="0 0 1"/>
+    </joint>
+    <link name="left_front_wheel">
+        <visual>
+            <geometry>
+                <cylinder radius="${wheel_radius}" length="${wheel_thickness}"/>
+            </geometry>
+            <material name="blue"/>
+        </visual>
+        <collision>
+            <geometry>
+                <cylinder radius="${wheel_radius}" length="${wheel_thickness}"/>
+            </geometry>
+        </collision>
+        <xacro:inertial_cylinder mass="${wheel_mass}" length="${wheel_thickness}" radius="${wheel_radius}">
+            <origin xyz="0 0 0" rpy="0 0 0"/>
+        </xacro:inertial_cylinder>
+    </link>
+    <gazebo reference="left_front_wheel">
+        <material>Gazebo/Blue</material>
+    </gazebo>
+    <!-- RIGHT FRONT WHEEL LINK -->
+    <joint name="right_front_wheel_joint" type="continuous">
+        <parent link="base_link"/>
+        <child link="right_front_wheel"/>
+        <origin xyz="${-wheel_offset_x} ${-wheel_offset_y} 0" rpy="${pi/2} 0 0"/>
+        <axis xyz="0 0 -1"/>
+    </joint>
+    <link name="right_front_wheel">
+        <visual>
+            <geometry>
+                <cylinder radius="${wheel_radius}" length="${wheel_thickness}"/>
+            </geometry>
+            <material name="blue"/>
+        </visual>
+        <collision>
+            <geometry>
+                <cylinder radius="${wheel_radius}" length="${wheel_thickness}"/>
+            </geometry>
+        </collision>
+        <xacro:inertial_cylinder mass="${wheel_mass}" length="${wheel_thickness}" radius="${wheel_radius}">
+            <origin xyz="0 0 0" rpy="0 0 0"/>
+        </xacro:inertial_cylinder>
+    </link>
+    <gazebo reference="right_front_wheel">
+        <material>Gazebo/Blue</material>
+    </gazebo>
+    <!-- LEFT REAR WHEEL LINK -->
+    <joint name="left_rear_wheel_joint" type="continuous">
+        <parent link="base_link"/>
+        <child link="left_rear_wheel"/>
+        <origin xyz="${wheel_offset_x} ${wheel_offset_y} 0" rpy="-${pi/2} 0 0"/>
+        <axis xyz="0 0 1"/>
+    </joint>
+    <link name="left_rear_wheel">
+        <visual>
+            <geometry>
+                <cylinder radius="${wheel_radius}" length="${wheel_thickness}"/>
+            </geometry>
+            <material name="blue"/>
+        </visual>
+        <collision>
+            <geometry>
+                <cylinder radius="${wheel_radius}" length="${wheel_thickness}"/>
+            </geometry>
+        </collision>
+        <xacro:inertial_cylinder mass="${wheel_mass}" length="${wheel_thickness}" radius="${wheel_radius}">
+            <origin xyz="0 0 0" rpy="0 0 0"/>
+        </xacro:inertial_cylinder>
+    </link>
+    <gazebo reference="left_rear_wheel">
+        <material>Gazebo/Blue</material>
+    </gazebo>
+    <!-- RIGHT REAR WHEEL LINK -->
+    <joint name="right_rear_wheel_joint" type="continuous">
+        <parent link="base_link"/>
+        <child link="right_rear_wheel"/>
+        <origin xyz="${wheel_offset_x} ${-wheel_offset_y} 0" rpy="${pi/2} 0 0"/>
+        <axis xyz="0 0 -1"/>
+    </joint>
+    <link name="right_rear_wheel">
+        <visual>
+            <geometry>
+                <cylinder radius="${wheel_radius}" length="${wheel_thickness}"/>
+            </geometry>
+            <material name="blue"/>
+        </visual>
+        <collision>
+            <geometry>
+                <cylinder radius="${wheel_radius}" length="${wheel_thickness}"/>
+            </geometry>
+        </collision>
+        <xacro:inertial_cylinder mass="${wheel_mass}" length="${wheel_thickness}" radius="${wheel_radius}">
+            <origin xyz="0 0 0" rpy="0 0 0"/>
+        </xacro:inertial_cylinder>
+    </link>
+    <gazebo reference=" right_rear_wheel">
+        <material>Gazebo/Blue</material>
+    </gazebo>
 </robot>
