Commit message: Pending changes exported from your codespace

File: description/camera.xacro (robot description, xacro)
@@ -4,5 +4,5 @@
         <parent link="chassis"/>
         <child link="camera_link"/>
-        <origin xyz="0.9 0 0.5" rpy="0 0.18 0"/>
+        <origin xyz="0.6 0 0.5" rpy="0 0.18 0"/>
     </joint>
     <link name="camera_link">

File: description/gazebo_control.xacro (robot description, xacro)
@@ -4,11 +4,7 @@
         <plugin name="diff_drive" filename="libgazebo_ros_diff_drive.so">
             <!-- Wheel Information -->
-            <left_joint>left_front_wheel_joint</left_joint>  <!-- Reference to the left front wheel joint -->
-            <right_joint>right_front_wheel_joint</right_joint>  <!-- Reference to the right front wheel joint -->
-            <wheel_separation>0.75</wheel_separation>  <!-- This can be adjusted to match your robot's wheelbase -->
-            <wheel_diameter>0.17</wheel_diameter>  <!-- Updated to match the wheel radius (2 * 0.085) -->
-            <left_joint>left_wheel_joint</left_joint>
-            <right_joint>right_wheel_joint</right_joint>
-            <wheel_separation>0.75</wheel_separation>
+             <left_joint>left_wheel_joint</left_joint>  <!-- Reference to the left front wheel joint -->
+            <right_joint>right_wheel_joint</right_joint>  <!-- Reference to the right front wheel joint -->
+            <wheel_separation>0.297</wheel_separation>
             <wheel_diameter>0.17</wheel_diameter>
             <!-- Limits -->

File: description/robot_core.xacro (robot description, xacro)
@@ -1,7 +1,7 @@
 <?xml version="1.0"?>
-<robot xmlns:xacro="http://www.ros.org/wiki/xacro">
+<robot xmlns:xacro="http://www.ros.org/wiki/xacro" >
     <xacro:include filename="inertial_macros.xacro"/>
-    <xacro:property name="chassis_length" value="1.02"/>  <!-- Updated length -->
-    <xacro:property name="chassis_width" value="0.70"/>   <!-- Updated width -->
+    <xacro:property name="chassis_length" value="0.7"/>  <!-- Updated length -->
+    <xacro:property name="chassis_width" value="0.5"/>   <!-- Updated width -->
     <xacro:property name="chassis_height" value="0.45"/>  <!-- Updated height -->
     <xacro:property name="chassis_mass" value="1.0"/>
@@ -9,7 +9,11 @@
     <xacro:property name="wheel_thickness" value="0.05"/>  <!-- Updated wheel thickness -->
     <xacro:property name="wheel_mass" value="0.05"/>
-    <xacro:property name="wheel_offset_x" value="0.51"/>   <!-- Updated offset for wheel placement -->
-    <xacro:property name="wheel_offset_y" value="0.375"/>   <!-- Updated offset for wheel placement -->
-    <xacro:property name="wheel_offset_z" value="0.0"/>    <!-- Height offset for wheels -->
+    <xacro:property name="wheel_offset_x" value="0.35"/>   <!-- Updated offset for wheel placement -->
+    <xacro:property name="wheel_offset_y" value="0.275"/>   <!-- Updated offset for wheel placement -->
+    <xacro:property name="wheel_offset_z" value="0.0"/>
+    <xacro:property name="caster_wheel_radius" value="0.085"/>
+    <xacro:property name="caster_wheel_mass" value="0.01"/>
+    <xacro:property name="caster_wheel_offset_x" value="0.075"/>
+    <xacro:property name="caster_wheel_offset_z" value="${wheel_offset_z - wheel_radius + caster_wheel_radius}"/>
     <material name="white">
         <color rgba="1 1 1 1" />
@@ -65,12 +69,12 @@
         <material>Gazebo/Orange</material>
     </gazebo>
-    <!-- LEFT FRONT WHEEL LINK -->
-    <joint name="left_front_wheel_joint" type="continuous">
+    <!-- LEFT WHEEL LINK -->
+    <joint name="left_wheel_joint" type="continuous">
         <parent link="base_link"/>
-        <child link="left_front_wheel"/>
-        <origin xyz="${-wheel_offset_x} ${wheel_offset_y} 0" rpy="-${pi/2} 0 0"/>
+        <child link="left_wheel"/>
+        <origin xyz="${wheel_offset_x} ${wheel_offset_y} 0" rpy="-${pi/2} 0 0"/>
         <axis xyz="0 0 1"/>
     </joint>
-    <link name="left_front_wheel">
+    <link name="left_wheel">
         <visual>
             <geometry>
@@ -81,5 +85,5 @@
         <collision>
             <geometry>
-                <cylinder radius="${wheel_radius}" length="${wheel_thickness}"/>
+                <sphere radius="${wheel_radius}"/>
             </geometry>
         </collision>
@@ -88,15 +92,15 @@
         </xacro:inertial_cylinder>
     </link>
-    <gazebo reference="left_front_wheel">
+    <gazebo reference="left_wheel">
         <material>Gazebo/Blue</material>
     </gazebo>
-    <!-- RIGHT FRONT WHEEL LINK -->
-    <joint name="right_front_wheel_joint" type="continuous">
+    <!-- RIGHT WHEEL LINK -->
+    <joint name="right_wheel_joint" type="continuous">
         <parent link="base_link"/>
-        <child link="right_front_wheel"/>
-        <origin xyz="${-wheel_offset_x} ${-wheel_offset_y} 0" rpy="${pi/2} 0 0"/>
+        <child link="right_wheel"/>
+        <origin xyz="${wheel_offset_x} ${-wheel_offset_y} 0" rpy="${pi/2} 0 0"/>
         <axis xyz="0 0 -1"/>
     </joint>
-    <link name="right_front_wheel">
+    <link name="right_wheel">
         <visual>
             <geometry>
@@ -107,5 +111,5 @@
         <collision>
             <geometry>
-                <cylinder radius="${wheel_radius}" length="${wheel_thickness}"/>
+                <sphere radius="${wheel_radius}"/>
             </geometry>
         </collision>
@@ -114,58 +118,33 @@
         </xacro:inertial_cylinder>
     </link>
-    <gazebo reference="right_front_wheel">
+    <gazebo reference="right_wheel">
         <material>Gazebo/Blue</material>
     </gazebo>
-    <!-- LEFT REAR WHEEL LINK -->
-    <joint name="left_rear_wheel_joint" type="continuous">
-        <parent link="base_link"/>
-        <child link="left_rear_wheel"/>
-        <origin xyz="${wheel_offset_x} ${wheel_offset_y} 0" rpy="-${pi/2} 0 0"/>
-        <axis xyz="0 0 1"/>
+    <!-- CASTER WHEEL LINK -->
+    <joint name="caster_wheel_joint" type="fixed">
+        <parent link="chassis"/>
+        <child link="caster_wheel"/>
+        <origin xyz="${caster_wheel_offset_x} 0 ${caster_wheel_offset_z}"/>
     </joint>
-    <link name="left_rear_wheel">
+    <link name="caster_wheel">
         <visual>
             <geometry>
-                <cylinder radius="${wheel_radius}" length="${wheel_thickness}"/>
+                <sphere radius="${caster_wheel_radius}"/>
             </geometry>
-            <material name="blue"/>
+            <material name="white"/>
         </visual>
         <collision>
             <geometry>
-                <cylinder radius="${wheel_radius}" length="${wheel_thickness}"/>
+                <sphere radius="${caster_wheel_radius}"/>
             </geometry>
         </collision>
-        <xacro:inertial_cylinder mass="${wheel_mass}" length="${wheel_thickness}" radius="${wheel_radius}">
+        <xacro:inertial_sphere mass="${caster_wheel_mass}" radius="${caster_wheel_radius}">
             <origin xyz="0 0 0" rpy="0 0 0"/>
-        </xacro:inertial_cylinder>
+        </xacro:inertial_sphere>
     </link>
-    <gazebo reference="left_rear_wheel">
-        <material>Gazebo/Blue</material>
-    </gazebo>
-    <!-- RIGHT REAR WHEEL LINK -->
-    <joint name="right_rear_wheel_joint" type="continuous">
-        <parent link="base_link"/>
-        <child link="right_rear_wheel"/>
-        <origin xyz="${wheel_offset_x} ${-wheel_offset_y} 0" rpy="${pi/2} 0 0"/>
-        <axis xyz="0 0 -1"/>
-    </joint>
-    <link name="right_rear_wheel">
-        <visual>
-            <geometry>
-                <cylinder radius="${wheel_radius}" length="${wheel_thickness}"/>
-            </geometry>
-            <material name="blue"/>
-        </visual>
-        <collision>
-            <geometry>
-                <cylinder radius="${wheel_radius}" length="${wheel_thickness}"/>
-            </geometry>
-        </collision>
-        <xacro:inertial_cylinder mass="${wheel_mass}" length="${wheel_thickness}" radius="${wheel_radius}">
-            <origin xyz="0 0 0" rpy="0 0 0"/>
-        </xacro:inertial_cylinder>
-    </link>
-    <gazebo reference=" right_rear_wheel">
-        <material>Gazebo/Blue</material>
+    <gazebo reference="caster_wheel">
+        <material>Gazebo/White</material>
+        <mu1 value="0.001"/>
+        <mu2 value="0.001"/>
     </gazebo>
 </robot>

File: description/ros2_control.xacro (robot description, xacro)
@@ -6,7 +6,5 @@
                 <plugin>diffdrive_arduino/DiffDriveArduino</plugin>
                 <param name="left_wheel_name">left_wheel_joint</param>
-                <param name="right_wheel_name">right_wheel_joint
-                <param name="left_front_wheel_name">left_front_wheel_joint</param>
-                <param name="right_front_wheel_name">right_front_wheel_joint</param>
+                <param name="right_wheel_name">right_wheel_joint</param>
                 <param name="loop_rate">30</param>
                 <param name="device">/dev/ttyUSB0</param>
@@ -24,20 +22,4 @@
             </joint>
             <joint name="right_wheel_joint">
-                <command_interface name="velocity">
-                    <param name="min">-10</param>
-                    <param name="max">10</param>
-                </command_interface>
-                <state_interface name="velocity"/>
-                <state_interface name="position"/>
-            </joint>
-            <joint name="left_front_wheel_joint">
-                <command_interface name="velocity">
-                    <param name="min">-10</param>
-                    <param name="max">10</param>
-                </command_interface>
-                <state_interface name="velocity"/>
-                <state_interface name="position"/>
-            </joint>
-            <joint name="right_front_wheel_joint">
                 <command_interface name="velocity">
                     <param name="min">-10</param>
@@ -70,20 +52,4 @@
                 <state_interface name="position"/>
             </joint>
-            <joint name="left_front_wheel_joint">
-                <command_interface name="velocity">
-                    <param name="min">-10</param>
-                    <param name="max">10</param>
-                </command_interface>
-                <state_interface name="velocity"/>
-                <state_interface name="position"/>
-            </joint>
-            <joint name="right_front_wheel_joint">
-                <command_interface name="velocity">
-                    <param name="min">-10</param>
-                    <param name="max">10</param>
-                </command_interface>
-                <state_interface name="velocity"/>
-                <state_interface name="position"/>
-            </joint>
         </ros2_control>
     </xacro:if>
